Commit message: Change variables to erlecopter

File: ardupilot_sitl_gazebo_plugin/urdf/erlecopter.xacro (robot description, xacro)
@@ -1,6 +1,6 @@
 <?xml version="1.0"?>
-<robot name="iris" xmlns:xacro="http://ros.org/wiki/xacro">
+<robot name="erlecopter" xmlns:xacro="http://ros.org/wiki/xacro">
   <!-- Properties -->
-  <xacro:property name="namespace" value="iris" />
+  <xacro:property name="namespace" value="erlecopter" />
   <xacro:property name="rotor_velocity_slowdown_sim" value="10" />
   <xacro:property name="mesh_file" value="erlecopter.dae" />
@@ -127,5 +127,4 @@
   <!-- Sonar height sensor -->
   <xacro:include filename="$(find ardupilot_sitl_gazebo_plugin)/urdf/sensors/sonar_sensor.urdf.xacro" />
- <!--
   <xacro:sonar_sensor
     name="sonar"
@@ -140,7 +139,6 @@
     <origin xyz="0.12 0.0 0.0" rpy="0 ${90*M_PI/180} 0"/>
   </xacro:sonar_sensor>
-     -->
     <!-- Frontal range sensor -->
- <!--  <xacro:sonar_sensor
+<!--  <xacro:sonar_sensor
     name="sonar2"
     parent="base_link"
@@ -155,5 +153,4 @@
   </xacro:sonar_sensor>
 -->
-<!--
   <xacro:include filename="$(find ardupilot_sitl_gazebo_plugin)/urdf/sensors/lidar_sensor.urdf.xacro" />
    <xacro:lidar_sensor
@@ -171,9 +168,8 @@
     <origin xyz="0.13 0.0 0.02" rpy="0 0 0"/>
   </xacro:lidar_sensor>
--->
   <!-- Downward facing camera -->
   <xacro:include filename="$(find ardupilot_sitl_gazebo_plugin)/urdf/sensors/generic_camera.urdf.xacro" />
   <xacro:generic_camera
-    name="iris/bottom"
+    name="erlecopter/bottom"
     parent="base_link"
     ros_topic="image_raw"
@@ -184,5 +180,5 @@
     image_format="R8G8B8"
     hfov="81"
-    framename="iris_bottomcam">
+    framename="erlecopter_bottomcam">
     <origin xyz="0.14 0.0 -0.02" rpy="0 ${M_PI/2} 0"/>
   </xacro:generic_camera>
@@ -190,5 +186,5 @@
   <xacro:include filename="$(find ardupilot_sitl_gazebo_plugin)/urdf/sensors/generic_camera.urdf.xacro" />
   <xacro:generic_camera
-    name="iris/front"
+    name="erlecopter/front"
     parent="base_link"
     ros_topic="image_front_raw"
@@ -199,5 +195,5 @@
     image_format="R8G8B8"
     hfov="81"
-    framename="iris_frontcam">
+    framename="erlecopter_frontcam">
     <origin xyz="0.17 0.0 0.0" rpy="0 0 0"/>
   </xacro:generic_camera>
@@ -218,5 +214,5 @@
     rotor_drag_coefficient="${rotor_drag_coefficient}"
     rolling_moment_coefficient="${rolling_moment_coefficient}"
-    mesh="iris_prop"
+    mesh="erlecopter_prop"
     mesh_scale="${mesh_scale_prop}"
     color="Yellow">
@@ -239,5 +235,5 @@
     rotor_drag_coefficient="${rotor_drag_coefficient}"
     rolling_moment_coefficient="${rolling_moment_coefficient}"
-    mesh="iris_prop"
+    mesh="erlecopter_prop"
     mesh_scale="${mesh_scale_prop}"
     color="Black">
@@ -259,5 +255,5 @@
     rotor_drag_coefficient="${rotor_drag_coefficient}"
     rolling_moment_coefficient="${rolling_moment_coefficient}"
-    mesh="iris_prop"
+    mesh="erlecopter_prop"
     mesh_scale="${mesh_scale_prop}"
     color="Yellow">
@@ -279,5 +275,5 @@
     rotor_drag_coefficient="${rotor_drag_coefficient}"
     rolling_moment_coefficient="${rolling_moment_coefficient}"
-    mesh="iris_prop"
+    mesh="erlecopter_prop"
     mesh_scale="${mesh_scale_prop}"
     color="Black">

File: ardupilot_sitl_gazebo_plugin/urdf/erlecopter_base.xacro (robot description, xacro)
@@ -1,6 +1,6 @@
 <?xml version="1.0"?>
-<robot name="iris" xmlns:xacro="http://ros.org/wiki/xacro">
+<robot name="erlecopter" xmlns:xacro="http://ros.org/wiki/xacro">
   <xacro:include filename="$(find rotors_description)/urdf/component_snippets.xacro" />
-  <!-- Instantiate iris "mechanics" -->
+  <!-- Instantiate erlecopter "mechanics" -->
   <xacro:include filename="$(find ardupilot_sitl_gazebo_plugin)/urdf/erlecopter.xacro" />
   <!-- Specify reference parameters for GNSS receiver. -->
