Commit message: Add Rover

File: ardupilot_sitl_gazebo_plugin/urdf/gps_home_location.xacro (robot description, xacro)
@@ -1,9 +1,9 @@
 <?xml version="1.0"?>
 <!-- File auto-generated by sim_vehicle.sh -->
-<!-- Location at Miramas -->
+<!-- Location at CMAC -->
 <robot xmlns:xacro="http://ros.org/wiki/xacro">
   <!-- The following GPS coordinates locate the center of Gazebo's map -->
-  <xacro:property name="referenceLatitude" value="44.1161693" />     <!-- in degrees -->
-  <xacro:property name="referenceLongitude" value="4.8427009" />   <!-- in degrees -->
-  <xacro:property name="referenceAltitude" value="103" />     <!-- in meters above sea level -->
+  <xacro:property name="referenceLatitude" value="-35.363261" />     <!-- in degrees -->
+  <xacro:property name="referenceLongitude" value="149.165230" />   <!-- in degrees -->
+  <xacro:property name="referenceAltitude" value="584" />     <!-- in meters above sea level -->
 </robot>
