Commit message: Change rover weight to avoid drifting

File: ardupilot_sitl_gazebo_plugin/urdf/rover.urdf (robot description, URDF)
Before this commit: robot rover, 7 links, 6 joints
Links:
- link chassis: mass 500.0 -> 800.0
- link front_left_wheel: mass 12 -> 20
- link front_right_wheel: mass 12 -> 20
- link rear_left_wheel: mass 12 -> 20
- link rear_right_wheel: mass 12 -> 20
