Commit message: GZ_REGISTER_WORLD_PLUGIN and Ardupilot 9002 & 9003 ports have been fixed

File: ardupilot_sitl_gazebo_rover_plugin/urdf/aircraft_base.xacro (robot description, xacro)
@@ -19,10 +19,10 @@
          <visual>
             <geometry>
-               <mesh filename="package://ardupilot_sitl_gazebo_plugin/meshes/meshes_drones/cessna/body.dae" />
-            </geometry>
-         </visual>
-         <collision name="collision">
-            <geometry>
-               <mesh filename="package://ardupilot_sitl_gazebo_plugin/meshes/meshes_drones/cessna/body.dae" />
+               <mesh filename="package://ardupilot_sitl_gazebo_rover_plugin/meshes/meshes_drones/cessna/body.dae" />
+            </geometry>
+         </visual>
+         <collision name="collision">
+            <geometry>
+               <mesh filename="package://ardupilot_sitl_gazebo_rover_plugin/meshes/meshes_drones/cessna/body.dae" />
             </geometry>
          </collision>
@@ -37,5 +37,5 @@
          <collision name="collision">
             <geometry>
-               <mesh filename="package://ardupilot_sitl_gazebo_plugin/meshes/meshes_drones/cessna/left_aileron.dae" />
+               <mesh filename="package://ardupilot_sitl_gazebo_rover_plugin/meshes/meshes_drones/cessna/left_aileron.dae" />
             </geometry>
             <origin xyz="1.92 -3.55 -1.3" rpy="-0.05 0 0.12" />
@@ -43,5 +43,5 @@
          <visual name="visual">
             <geometry>
-               <mesh filename="package://ardupilot_sitl_gazebo_plugin/meshes/meshes_drones/cessna/left_aileron.dae" />
+               <mesh filename="package://ardupilot_sitl_gazebo_rover_plugin/meshes/meshes_drones/cessna/left_aileron.dae" />
             </geometry>
             <origin xyz="1.92 -3.55 -1.3" rpy="-0.05 0 0.12" />
@@ -66,5 +66,5 @@
          <collision name="collision">
             <geometry>
-               <mesh filename="package://ardupilot_sitl_gazebo_plugin/meshes/meshes_drones/cessna/right_aileron.dae" />
+               <mesh filename="package://ardupilot_sitl_gazebo_rover_plugin/meshes/meshes_drones/cessna/right_aileron.dae" />
             </geometry>
             <origin xyz="1.92 3.57 -1.3" rpy="0.05 0 -0.12" />
@@ -72,5 +72,5 @@
          <visual name="visual">
             <geometry>
-               <mesh filename="package://ardupilot_sitl_gazebo_plugin/meshes/meshes_drones/cessna/right_aileron.dae" />
+               <mesh filename="package://ardupilot_sitl_gazebo_rover_plugin/meshes/meshes_drones/cessna/right_aileron.dae" />
             </geometry>
             <origin xyz="1.92 3.57 -1.3" rpy="0.05 0 -0.12" />
@@ -95,5 +95,5 @@
          <collision name="collision">
             <geometry>
-               <mesh filename="package://ardupilot_sitl_gazebo_plugin/meshes/meshes_drones/cessna/left_flap.dae" />
+               <mesh filename="package://ardupilot_sitl_gazebo_rover_plugin/meshes/meshes_drones/cessna/left_flap.dae" />
             </geometry>
             <origin xyz="1.60 -1.58 -1.42" rpy="-0.02 0 -0.02" />
@@ -101,5 +101,5 @@
          <visual name="visual">
             <geometry>
-               <mesh filename="package://ardupilot_sitl_gazebo_plugin/meshes/meshes_drones/cessna/left_flap.dae" />
+               <mesh filename="package://ardupilot_sitl_gazebo_rover_plugin/meshes/meshes_drones/cessna/left_flap.dae" />
             </geometry>
             <origin xyz="1.60 -1.58 -1.42" rpy="-0.02 0 -0.02" />
@@ -124,5 +124,5 @@
          <collision name="collision">
             <geometry>
-               <mesh filename="package://ardupilot_sitl_gazebo_plugin/meshes/meshes_drones/cessna/right_flap.dae" />
+               <mesh filename="package://ardupilot_sitl_gazebo_rover_plugin/meshes/meshes_drones/cessna/right_flap.dae" />
             </geometry>
             <origin xyz="1.62 1.54 -1.46" rpy="-0.02 0 0.02" />
@@ -130,5 +130,5 @@
          <visual name="visual">
             <geometry>
-               <mesh filename="package://ardupilot_sitl_gazebo_plugin/meshes/meshes_drones/cessna/right_flap.dae" />
+               <mesh filename="package://ardupilot_sitl_gazebo_rover_plugin/meshes/meshes_drones/cessna/right_flap.dae" />
             </geometry>
             <origin xyz="1.62 1.54 -1.46" rpy="-0.02 0 0.02" />
@@ -153,5 +153,5 @@
          <collision name="collision">
             <geometry>
-               <mesh filename="package://ardupilot_sitl_gazebo_plugin/meshes/meshes_drones/cessna/elevators.dae" />
+               <mesh filename="package://ardupilot_sitl_gazebo_rover_plugin/meshes/meshes_drones/cessna/elevators.dae" />
             </geometry>
             <origin xyz="5.55 0 -0.57" rpy="0 0 0" />
@@ -159,5 +159,5 @@
          <visual name="visual">
             <geometry>
-               <mesh filename="package://ardupilot_sitl_gazebo_plugin/meshes/meshes_drones/cessna/elevators.dae" />
+               <mesh filename="package://ardupilot_sitl_gazebo_rover_plugin/meshes/meshes_drones/cessna/elevators.dae" />
             </geometry>
             <origin xyz="5.55 0 -0.57" rpy="0 0 0" />
@@ -182,5 +182,5 @@
          <collision name="collision">
             <geometry>
-               <mesh filename="package://ardupilot_sitl_gazebo_plugin/meshes/meshes_drones/cessna/rudder.dae" />
+               <mesh filename="package://ardupilot_sitl_gazebo_rover_plugin/meshes/meshes_drones/cessna/rudder.dae" />
             </geometry>
             <origin xyz="5.1 0 -3.25" rpy="0 0.35 0" />
@@ -188,5 +188,5 @@
          <visual name="visual">
             <geometry>
-               <mesh filename="package://ardupilot_sitl_gazebo_plugin/meshes/meshes_drones/cessna/rudder.dae" />
+               <mesh filename="package://ardupilot_sitl_gazebo_rover_plugin/meshes/meshes_drones/cessna/rudder.dae" />
             </geometry>
             <origin xyz="5.1 0 -3.25" rpy="0 0.35 0" />
@@ -211,10 +211,10 @@
          <collision name="collision">
             <!--<geometry>
-               <mesh filename="package://ardupilot_sitl_gazebo_plugin/meshes/meshes_drones/cessna/cessna_prop.dae" />
+               <mesh filename="package://ardupilot_sitl_gazebo_rover_plugin/meshes/meshes_drones/cessna/cessna_prop.dae" />
             </geometry>-->
          </collision>
          <visual name="visual">
             <geometry>
-               <mesh filename="package://ardupilot_sitl_gazebo_plugin/meshes/meshes_drones/cessna/cessna_prop.dae" />
+               <mesh filename="package://ardupilot_sitl_gazebo_rover_plugin/meshes/meshes_drones/cessna/cessna_prop.dae" />
             </geometry>
          </visual>
@@ -244,5 +244,5 @@
          <visual name="visual">
             <geometry>
-               <mesh filename="package://ardupilot_sitl_gazebo_plugin/meshes/meshes_drones/cessna/cessna_front_wheel.dae" />
+               <mesh filename="package://ardupilot_sitl_gazebo_rover_plugin/meshes/meshes_drones/cessna/cessna_front_wheel.dae" />
             </geometry>
             <origin xyz="-0.712 0 0.313" rpy="0 0 0" />
@@ -273,5 +273,5 @@
          <visual name="visual">
             <geometry>
-               <mesh filename="package://ardupilot_sitl_gazebo_plugin/meshes/meshes_drones/cessna/cessna_rear_left_wheel.dae" />
+               <mesh filename="package://ardupilot_sitl_gazebo_rover_plugin/meshes/meshes_drones/cessna/cessna_rear_left_wheel.dae" />
             </geometry>
             <origin xyz="1 1.27 0.25" rpy="0 0 0" />
@@ -302,5 +302,5 @@
          <visual name="visual">
             <geometry>
-               <mesh filename="package://ardupilot_sitl_gazebo_plugin/meshes/meshes_drones/cessna/cessna_rear_right_wheel.dae" />
+               <mesh filename="package://ardupilot_sitl_gazebo_rover_plugin/meshes/meshes_drones/cessna/cessna_rear_right_wheel.dae" />
             </geometry>
             <origin xyz="1 -1.27 0.25" rpy="0 0 0" />
@@ -403,5 +403,5 @@
       </gazebo>
       <gazebo>
-         <plugin name="left_wing" filename="libliftdrag_plugin.so">
+         <plugin name="left_wing" filename="libliftdrag_rover_plugin.so">
             <a0>0.0598</a0>
             <cla>4.752798721</cla>
@@ -423,5 +423,5 @@
       </gazebo>
       <gazebo>
-         <plugin name="right_wing" filename="libliftdrag_plugin.so">
+         <plugin name="right_wing" filename="libliftdrag_rover_plugin.so">
             <a0>0.0598</a0>
             <cla>4.752798721</cla>
@@ -443,5 +443,5 @@
       </gazebo>
       <gazebo>
-         <plugin name="left_flap_wing" filename="libliftdrag_plugin.so">
+         <plugin name="left_flap_wing" filename="libliftdrag_rover_plugin.so">
             <a0>0.0598</a0>
             <cla>4.752798721</cla>
@@ -464,5 +464,5 @@
       </gazebo>
       <gazebo>
-         <plugin name="right_flap_wing" filename="libliftdrag_plugin.so">
+         <plugin name="right_flap_wing" filename="libliftdrag_rover_plugin.so">
             <a0>0.0598</a0> <!-- -3.2 deg (0.09:5deg, 0.17:10deg)-->
             <cla>4.752798721</cla>
@@ -484,5 +484,5 @@
       </gazebo>
       <gazebo>
-         <plugin name="elevator" filename="libliftdrag_plugin.so">
+         <plugin name="elevator" filename="libliftdrag_rover_plugin.so">
             <a0>-0.2</a0>
             <cla>4.752798721</cla>
@@ -504,5 +504,5 @@
       </gazebo>
       <gazebo>
-         <plugin name="rudder" filename="libliftdrag_plugin.so">
+         <plugin name="rudder" filename="libliftdrag_rover_plugin.so">
             <a0>0</a0>
             <cla>4.752798721</cla>
@@ -524,5 +524,5 @@
       </gazebo>
       <gazebo>
-         <plugin name="propeller_top_blade" filename="libliftdrag_plugin.so">
+         <plugin name="propeller_top_blade" filename="libliftdrag_rover_plugin.so">
             <a0>0.4</a0>
             <cla>4.752798721</cla>
@@ -542,5 +542,5 @@
       </gazebo>
       <gazebo>
-         <plugin name="propeller_bottom_blade" filename="libliftdrag_plugin.so">
+         <plugin name="propeller_bottom_blade" filename="libliftdrag_rover_plugin.so">
             <a0>0.4</a0>
             <cla>4.752798721</cla>

File: ardupilot_sitl_gazebo_rover_plugin/urdf/cessna.xacro (robot description, xacro)
@@ -3,9 +3,9 @@
    <!-- Properties -->
    <xacro:property name="namespace" value="cessna" />
-   <xacro:include filename="$(find ardupilot_sitl_gazebo_plugin)/urdf/aircraft_base.xacro" />
+   <xacro:include filename="$(find ardupilot_sitl_gazebo_rover_plugin)/urdf/aircraft_base.xacro" />
    <!-- Instantiate aircraft_base_macro once -->
    <xacro:aircraft_base_macro />
    <xacro:property name="M_PI" value="3.1415926535897931" />
-   <xacro:include filename="$(find ardupilot_sitl_gazebo_plugin)/urdf/recorder_camera.xacro" />
+   <xacro:include filename="$(find ardupilot_sitl_gazebo_rover_plugin)/urdf/recorder_camera.xacro" />
    <!--
    <xacro:recorder_camera name="recorder_cam_front_with_uav"

File: ardupilot_sitl_gazebo_rover_plugin/urdf/cessna_base.xacro (robot description, xacro)
@@ -3,7 +3,7 @@
    <xacro:include filename="$(find rotors_description)/urdf/component_snippets.xacro" />
    <!-- Instantiate iris "mechanics" -->
-   <xacro:include filename="$(find ardupilot_sitl_gazebo_plugin)/urdf/cessna.xacro" />
+   <xacro:include filename="$(find ardupilot_sitl_gazebo_rover_plugin)/urdf/cessna.xacro" />
    <!-- Specify reference parameters for GNSS receiver. -->
-   <xacro:include filename="$(find ardupilot_sitl_gazebo_plugin)/urdf/gps_home_location.xacro" />
+   <xacro:include filename="$(find ardupilot_sitl_gazebo_rover_plugin)/urdf/gps_home_location.xacro" />
    <!-- Reference heading is equivalent to rotating Gazebo's map. We do not use it for we would loose the match X=North, Y=West -->
    <!-- in degrees, 0 so North is towards positive X values, and East is towards negative Y values -->

File: ardupilot_sitl_gazebo_rover_plugin/urdf/erlecopter.xacro (robot description, xacro)
@@ -43,5 +43,5 @@
   <!-- Included URDF Files -->
   <!-- <xacro:include filename="$(find rotors_description)/urdf/multirotor_base.xacro" /> -->
-  <xacro:include filename="$(find ardupilot_sitl_gazebo_plugin)/urdf/multirotor_base.xacro" />
+  <xacro:include filename="$(find ardupilot_sitl_gazebo_rover_plugin)/urdf/multirotor_base.xacro" />
   <!-- Instantiate multirotor_base_macro once -->
   <xacro:multirotor_base_macro
@@ -59,5 +59,5 @@
   <xacro:property name="M_PI" value="3.1415926535897931" />
   <!-- Recorder cameras -->
-  <xacro:include filename="$(find ardupilot_sitl_gazebo_plugin)/urdf/recorder_camera.xacro" />
+  <xacro:include filename="$(find ardupilot_sitl_gazebo_rover_plugin)/urdf/recorder_camera.xacro" />
   <!--
 <xacro:recorder_camera
@@ -126,5 +126,5 @@
   <!-- Recorder cameras END -->
   <!-- Sonar height sensor -->
-  <xacro:include filename="$(find ardupilot_sitl_gazebo_plugin)/urdf/sensors/sonar_sensor.urdf.xacro" />
+  <xacro:include filename="$(find ardupilot_sitl_gazebo_rover_plugin)/urdf/sensors/sonar_sensor.urdf.xacro" />
   <xacro:sonar_sensor
     name="sonar"
@@ -153,5 +153,5 @@
   </xacro:sonar_sensor>
 -->
-  <xacro:include filename="$(find ardupilot_sitl_gazebo_plugin)/urdf/sensors/lidar_sensor.urdf.xacro" />
+  <xacro:include filename="$(find ardupilot_sitl_gazebo_rover_plugin)/urdf/sensors/lidar_sensor.urdf.xacro" />
    <xacro:lidar_sensor
     name="sonar2"
@@ -169,5 +169,5 @@
   </xacro:lidar_sensor>
 <!-- Prasad N R Downward facing camera
-  <xacro:include filename="$(find ardupilot_sitl_gazebo_plugin)/urdf/sensors/generic_camera.urdf.xacro" />
+  <xacro:include filename="$(find ardupilot_sitl_gazebo_rover_plugin)/urdf/sensors/generic_camera.urdf.xacro" />
   <xacro:generic_camera
     name="erlecopter/bottom"
@@ -185,5 +185,5 @@
 -->
   <!-- Front facing camera 320 x 240 @ 5Hz instead of 640x360 @ 25Hz-->
-  <xacro:include filename="$(find ardupilot_sitl_gazebo_plugin)/urdf/sensors/generic_camera.urdf.xacro" />
+  <xacro:include filename="$(find ardupilot_sitl_gazebo_rover_plugin)/urdf/sensors/generic_camera.urdf.xacro" />
   <xacro:generic_camera
     name="erlecopter/front"

File: ardupilot_sitl_gazebo_rover_plugin/urdf/erlecopter_base.xacro (robot description, xacro)
@@ -3,7 +3,7 @@
   <xacro:include filename="$(find rotors_description)/urdf/component_snippets.xacro" />
   <!-- Instantiate erlecopter "mechanics" -->
-  <xacro:include filename="$(find ardupilot_sitl_gazebo_plugin)/urdf/erlecopter.xacro" />
+  <xacro:include filename="$(find ardupilot_sitl_gazebo_rover_plugin)/urdf/erlecopter.xacro" />
   <!-- Specify reference parameters for GNSS receiver. -->
-  <xacro:include filename="$(find ardupilot_sitl_gazebo_plugin)/urdf/gps_home_location.xacro" />
+  <xacro:include filename="$(find ardupilot_sitl_gazebo_rover_plugin)/urdf/gps_home_location.xacro" />
   <!-- Reference heading is equivalent to rotating Gazebo's map.
        We do not use it for we would loose the match X=North, Y=West -->

File: ardupilot_sitl_gazebo_rover_plugin/urdf/iris.xacro (robot description, xacro)
@@ -43,5 +43,5 @@
   <!-- Included URDF Files -->
   <!-- <xacro:include filename="$(find rotors_description)/urdf/multirotor_base.xacro" /> -->
-  <xacro:include filename="$(find ardupilot_sitl_gazebo_plugin)/urdf/multirotor_base.xacro" />
+  <xacro:include filename="$(find ardupilot_sitl_gazebo_rover_plugin)/urdf/multirotor_base.xacro" />
   <!-- Instantiate multirotor_base_macro once -->
   <xacro:multirotor_base_macro
@@ -59,5 +59,5 @@
   <xacro:property name="M_PI" value="3.1415926535897931" />
   <!-- Recorder cameras -->
-  <xacro:include filename="$(find ardupilot_sitl_gazebo_plugin)/urdf/recorder_camera.xacro" />
+  <xacro:include filename="$(find ardupilot_sitl_gazebo_rover_plugin)/urdf/recorder_camera.xacro" />
   <!--
 <xacro:recorder_camera
@@ -126,5 +126,5 @@
   <!-- Recorder cameras END -->
   <!-- Sonar height sensor -->
-  <xacro:include filename="$(find ardupilot_sitl_gazebo_plugin)/urdf/sensors/sonar_sensor.urdf.xacro" />
+  <xacro:include filename="$(find ardupilot_sitl_gazebo_rover_plugin)/urdf/sensors/sonar_sensor.urdf.xacro" />
  <!--
   <xacro:sonar_sensor
@@ -156,5 +156,5 @@
 -->
 <!--
-  <xacro:include filename="$(find ardupilot_sitl_gazebo_plugin)/urdf/sensors/lidar_sensor.urdf.xacro" />
+  <xacro:include filename="$(find ardupilot_sitl_gazebo_rover_plugin)/urdf/sensors/lidar_sensor.urdf.xacro" />
    <xacro:lidar_sensor
     name="sonar2"
@@ -173,5 +173,5 @@
 -->
   <!-- Downward facing camera -->
-  <xacro:include filename="$(find ardupilot_sitl_gazebo_plugin)/urdf/sensors/generic_camera.urdf.xacro" />
+  <xacro:include filename="$(find ardupilot_sitl_gazebo_rover_plugin)/urdf/sensors/generic_camera.urdf.xacro" />
   <xacro:generic_camera
     name="iris/bottom"
@@ -188,5 +188,5 @@
   </xacro:generic_camera>
   <!-- Front facing camera -->
-  <xacro:include filename="$(find ardupilot_sitl_gazebo_plugin)/urdf/sensors/generic_camera.urdf.xacro" />
+  <xacro:include filename="$(find ardupilot_sitl_gazebo_rover_plugin)/urdf/sensors/generic_camera.urdf.xacro" />
   <xacro:generic_camera
     name="iris/front"

File: ardupilot_sitl_gazebo_rover_plugin/urdf/iris_base.xacro (robot description, xacro)
@@ -3,7 +3,7 @@
   <xacro:include filename="$(find rotors_description)/urdf/component_snippets.xacro" />
   <!-- Instantiate iris "mechanics" -->
-  <xacro:include filename="$(find ardupilot_sitl_gazebo_plugin)/urdf/iris.xacro" />
+  <xacro:include filename="$(find ardupilot_sitl_gazebo_rover_plugin)/urdf/iris.xacro" />
   <!-- Specify reference parameters for GNSS receiver. -->
-  <xacro:include filename="$(find ardupilot_sitl_gazebo_plugin)/urdf/gps_home_location.xacro" />
+  <xacro:include filename="$(find ardupilot_sitl_gazebo_rover_plugin)/urdf/gps_home_location.xacro" />
   <!-- Reference heading is equivalent to rotating Gazebo's map.
        We do not use it for we would loose the match X=North, Y=West -->

File: ardupilot_sitl_gazebo_rover_plugin/urdf/multirotor_base.xacro (robot description, xacro)
@@ -49,5 +49,5 @@
         <origin xyz="0 0 0" rpy="0 0 0" />
         <geometry>
-          <mesh filename="package://ardupilot_sitl_gazebo_plugin/meshes/meshes_drones/${mesh_file}"
+          <mesh filename="package://ardupilot_sitl_gazebo_rover_plugin/meshes/meshes_drones/${mesh_file}"
             scale="${mesh_scale}" />
           <!-- <box size="${body_width} ${body_width} ${body_height}"/> --> <!-- [m] [m] [m] -->
@@ -97,5 +97,5 @@
           <!-- <cylinder length="0.005" radius="${radius_rotor}"/> --> <!-- [m] -->
           <!-- <mesh filename="package://rotors_description/meshes/propeller_${direction}.dae" -->
-          <mesh filename="package://ardupilot_sitl_gazebo_plugin/meshes/meshes_drones/${mesh}_${direction}.dae"
+          <mesh filename="package://ardupilot_sitl_gazebo_rover_plugin/meshes/meshes_drones/${mesh}_${direction}.dae"
             scale="${mesh_scale}" />
           <!-- <box size="${2*radius_rotor} 0.01 0.005"/> -->

File: ardupilot_sitl_gazebo_rover_plugin/urdf/rover.urdf (robot description, URDF)
Before this commit: robot rover, 7 links, 6 joints
Links:
- link chassis: geometry collision box size=1.34 1.0 0.06; visual mesh filename=package://ardupilot_sitl_gazebo_rover_plugin/meshes/meshes_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 scale=0.0055 0.0055 0.0055
- link front_left_wheel: geometry collision cylinder length=0.2794 radius=0.3175; visual mesh filename=package://ardupilot_sitl_gazebo_rover_plugin/meshes/meshes_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 scale=0.007 0.007 0.007
- link front_right_wheel: geometry collision cylinder length=0.2794 radius=0.3175; visual mesh filename=package://ardupilot_sitl_gazebo_rover_plugin/meshes/meshes_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 scale=0.007 0.007 0.007
- link rear_left_wheel: geometry collision cylinder length=0.2794 radius=0.3175; visual mesh filename=package://ardupilot_sitl_gazebo_rover_plugin/meshes/meshes_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 scale=0.007 0.007 0.007
- link rear_right_wheel: geometry collision cylinder length=0.2794 radius=0.3175; visual mesh filename=package://ardupilot_sitl_gazebo_rover_plugin/meshes/meshes_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 scale=0.007 0.007 0.007

File: ardupilot_sitl_gazebo_rover_plugin/urdf/rover_scaled.urdf (robot description, URDF)
Before this commit: robot rover, 7 links, 6 joints
Links:
- link chassis: geometry collision box size=0.268 0.2 0.012; visual mesh filename=package://ardupilot_sitl_gazebo_rover_plugin/meshes/meshes_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 scale=0.0011 0.0011 0.0011
- link front_left_wheel: geometry collision cylinder length=0.05588 radius=0.0635; visual mesh filename=package://ardupilot_sitl_gazebo_rover_plugin/meshes/meshes_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 scale=0.0014 0.0014 0.0014
- link front_right_wheel: geometry collision cylinder length=0.05588 radius=0.0635; visual mesh filename=package://ardupilot_sitl_gazebo_rover_plugin/meshes/meshes_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 scale=0.0014 0.0014 0.0014
- link rear_left_wheel: geometry collision cylinder length=0.05588 radius=0.0635; visual mesh filename=package://ardupilot_sitl_gazebo_rover_plugin/meshes/meshes_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 scale=0.0014 0.0014 0.0014
- link rear_right_wheel: geometry collision cylinder length=0.05588 radius=0.0635; visual mesh filename=package://ardupilot_sitl_gazebo_rover_plugin/meshes/meshes_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 scale=0.0014 0.0014 0.0014

File: ardupilot_sitl_gazebo_rover_plugin/urdf/sensors/kinect.urdf.xacro (robot description, xacro)
@@ -31,5 +31,5 @@
        <origin xyz="0 0 0" rpy="0 0 ${M_PI/2}"/>
         <geometry>
-         <mesh filename="package://ardupilot_sitl_gazebo_plugin/meshes/meshes_sensors/kinect/kinect.dae"/>
+         <mesh filename="package://ardupilot_sitl_gazebo_rover_plugin/meshes/meshes_sensors/kinect/kinect.dae"/>
         </geometry>
       </visual>

File: ardupilot_sitl_gazebo_rover_plugin/urdf/sensors/lidar_sensor.urdf.xacro (robot description, xacro)
@@ -18,6 +18,6 @@
           <!--<box size="0.01 0.01 0.01" /> -->
           <!-- <mesh filename="package://rotors_description/meshes/sonar_sensor/max_sonar_ez4.dae"/> -->
-           <!--<mesh filename="package://ardupilot_sitl_gazebo_plugin/meshes/${sensor_mesh}"/>-->
-         <!-- <mesh filename="package://ardupilot_sitl_gazebo_plugin/meshes/lidar_lite_v2/meshes/lidar_lite_v2.dae"/> -->
+           <!--<mesh filename="package://ardupilot_sitl_gazebo_rover_plugin/meshes/${sensor_mesh}"/>-->
+         <!-- <mesh filename="package://ardupilot_sitl_gazebo_rover_plugin/meshes/lidar_lite_v2/meshes/lidar_lite_v2.dae"/> -->
         </geometry>
       </visual>

File: ardupilot_sitl_gazebo_rover_plugin/urdf/sensors/sonar_sensor.urdf.xacro (robot description, xacro)
@@ -18,7 +18,7 @@
           <!--<box size="0.01 0.01 0.01" /> -->
           <!-- <mesh filename="package://rotors_description/meshes/sonar_sensor/max_sonar_ez4.dae"/> -->
-           <!--<mesh filename="package://ardupilot_sitl_gazebo_plugin/meshes/${sensor_mesh}"/>-->
+           <!--<mesh filename="package://ardupilot_sitl_gazebo_rover_plugin/meshes/${sensor_mesh}"/>-->
            <mesh filename="model://${sensor_mesh}"/>
-         <!-- <mesh filename="package://ardupilot_sitl_gazebo_plugin/meshes/lidar_lite_v2/meshes/lidar_lite_v2.dae"/> -->
+         <!-- <mesh filename="package://ardupilot_sitl_gazebo_rover_plugin/meshes/lidar_lite_v2/meshes/lidar_lite_v2.dae"/> -->
         </geometry>
       </visual>
